File: icetest.sch (KiCad schematic (older format))
At the start: 30 parts

Commit message: more layout
Parts:
- W12: value TEST_1P -> +1.2
Changed lines of the file:
@@
 P 7000 2000
 F 0 "W12" H 7000 2270 50  0000 C CNN
-F 1 "TEST_1P" H 7000 2200 50  0000 C CNN
+F 1 "+1.2" H 7000 2200 50  0000 C CNN
 F 2 "Measurement_Points:Measurement_Point_Square-SMD-Pad_Small" H 7200 2000 50  0001 C CNN
 F 3 "" H 7200 2000 50  0000 C CNN
