File: icedaq/icedaq-analog.sch (KiCad schematic (older format))
At the start: 3 parts, among them U2 iCE40HX1K-VQ100

Commit message: update
Parts:
- added U?: LM324, symbol LM324
Changed lines of the file:
@@
+	1    0    0    -1
+$EndComp
+$Comp
+L LM324 U?
+U 1 1 586176AF
+P 6500 1950
+F 0 "U?" H 6550 2150 50  0000 C CNN
+F 1 "LM324" H 6650 1750 50  0000 C CNN
+F 2 "" H 6450 2050 50  0000 C CNN
+F 3 "" H 6550 2150 50  0000 C CNN
+	1    6500 1950
 	1    0    0    -1
 $EndComp

Commit message: icedaq: update
Parts:
- removed unit 3 of U2
- removed unit 6 of U2
- removed U?: LM324, symbol LM324
- added D1, D2, D3, D4, D5, D6, D7, D8: D_Small, local:D_0603_HandSoldering, symbol D_Small
- added DAC1, DAC2: DACx311, local:SC70, symbol DACx311
- added J1: analog outputs, Terminal_Blocks:TerminalBlock_Pheonix_MPT-2.54mm_4pol, symbol Screw_Terminal_1x04
- added J2: analog inputs, Terminal_Blocks:TerminalBlock_Pheonix_MPT-2.54mm_6pol, symbol Screw_Terminal_1x06
- added R1: 10k, Resistors_SMD:R_0603_HandSoldering, symbol R
- added R10, R11, R12, R16, R2, R20, R21, R22, R23, R9: R, Resistors_SMD:R_0603_HandSoldering, symbol R
- added R13, R14, R15, R17, R18, R19, R3, R4, R5, R6, R7, R8: 1k, Resistors_SMD:R_0603_HandSoldering, symbol R
- added U4: oscillator4, local:OSC_SMD_1, symbol oscillator4
- added U7: MCP6004, local:SOIC-14, symbol MCP6004
- U2: footprint (none) -> local:VQFP-100
- U5, U6: renamed from U?; footprint (none) -> local:VSSOP-8
Connections:
- net labels added: +5V, clk, cs1, cs2, din1, din2, din3, din4, dout1, dout2, in1, in1a, in2a, in3, in3a, in4a, out3, out3a, out4, out4a, sclk1, sclk2, sclk4, slkc3, sync3, sync4
- wire segments 0 -> 109
- no-connect marks 0 -> 4
Other:
- note added: "input buffer, then divide 5V -> 3.3V"
- note added: "output buffer amplifies 3.3V -> 5V"
- moved on the sheet: U2D, U5, U6

Commit message: icedaq layout
Parts:
- removed R1: 10k, Resistors_SMD:R_0603_HandSoldering, symbol R
- removed U4: oscillator4, local:OSC_SMD_1, symbol oscillator4
- added CD11, CD12, CD13, CD6, CD7: C_Small, Capacitors_SMD:C_0603_HandSoldering, symbol C_Small
- added unit 3 of U2
Connections:
- net labels added: GCLK2
- wire segments 109 -> 107
- no-connect marks 4 -> 21
Other:
- moved on the sheet: DAC1, DAC2

Commit message: minor
Other:
- note added: "gain=1 input buffer, then divide 5V -> 3.3V"
- note added: "non-inverting gain=1.5, output buffer amplifies 3.3V -> 5V"
- note removed: "input buffer, then divide 5V -> 3.3V"
- note removed: "output buffer amplifies 3.3V -> 5V"
Changed lines of the file:
@@
 	6150 2250 6150 2200
 Text Notes 7300 650  0    60   ~ 0
-input buffer, then divide 5V -> 3.3V
+gain=1 input buffer, then divide 5V -> 3.3V
 $Comp
 L MCP6004 U7
@@
 out3a
 Text Notes 6200 4250 0    60   ~ 0
-output buffer amplifies 3.3V -> 5V
+non-inverting gain=1.5, output buffer amplifies 3.3V -> 5V
 $Comp
 L +5V #PWR065
@@
 P 10450 3200
 F 0 "J2" H 10450 3850 50  0000 C TNN
-F 1 "analog inputs" V 10300 3200 50  0000 C TNN
+F 1 "analog inputs" H 10550 3950 50  0000 C TNN
 F 2 "Terminal_Blocks:TerminalBlock_Pheonix_MPT-2.54mm_6pol" H 10450 2575 50  0001 C CNN
 F 3 "" H 10425 3600 50  0001 C CNN
@@
 P 7300 3450
 F 0 "J1" H 7300 3900 50  0000 C TNN
-F 1 "analog outputs" V 7150 3450 50  0000 C TNN
+F 1 "analog outputs" H 7400 4050 50  0000 C TNN
 F 2 "Terminal_Blocks:TerminalBlock_Pheonix_MPT-2.54mm_4pol" H 7300 3025 50  0001 C CNN
 F 3 "" H 7275 3650 50  0001 C CNN

Commit message: icedaq: change input filter
Parts:
- removed D1, D2, D3, D4, D5, D6, D7, D8: D_Small, local:D_0603_HandSoldering, symbol D_Small
- added R24, R25, R26, R27: R, Resistors_SMD:R_0603_HandSoldering, symbol R
- R13, R14: value 1k -> R
- R21, R23: value R -> 1k
Connections:
- wire segments 107 -> 89
Other:
- moved on the sheet: R10, R12

Commit message: icedaq: update
Parts:
- removed J2: analog inputs, Terminal_Blocks:TerminalBlock_Pheonix_MPT-2.54mm_6pol, symbol Screw_Terminal_1x06
- added J2: analog inputs, Terminal_Blocks:TerminalBlock_Pheonix_MPT-2.54mm_4pol, symbol Screw_Terminal_1x04
Connections:
- net labels added: MISO1, MOSI1, SCLK1, SS1, cs5, cs6, din5, din6, dout5, dout6, sclk5, sclk6
- net labels removed: GCLK2, cs1, cs2, din1, din2, dout1, dout2, in2a, in4a, sclk1, sclk2
- wire segments 89 -> 88
- no-connect marks 21 -> 20
Other:
- note added: "ADCs"
- note added: "DACs"
- moved on the sheet: CD11, CD6, CD7
